File: Mini-Lora-Grove.brd (EAGLE design)
At the start: 68.8 x 25.7 mm, 24 parts, among them P1 GND, P2 PADNORMAL, P3 PADNORMAL, P4 PADNORMAL, U1 24AA02E64T

Commit message: Bump to V1.1a
Parts:
- removed P2, P3: PADNORMAL, _c2h:PAD
Connections:
- net SCL: now also U$6.A5-1; no longer P3.1
- net SDA: now also U$6.A4-1; no longer P2.1
Routing:
- net SDA: track 26.3 -> 51.3 mm
- net SCL: track 26.9 -> 41.4 mm
Other:
- board text added: "Mini-Lora V1.1a"
- board text added: "V1.1a"
- board text removed: "Mini-Lora V1.1"
- board text removed: "V1.1"
