File: Mini-Lora-Grove.sch (EAGLE design)
At the start: 22 parts, among them P1 GND, P2 PADNORMAL, P3 PADNORMAL, P4 PADNORMAL, U1 24AA02E64T

Commit message: Bump to V1.1a
Parts:
- removed P2, P3: PADNORMAL, _c2h:PADNORMAL
Connections:
- net SCL: now also U$6.A5-1; no longer P3.1
- net SDA: now also U$6.A4-1; no longer P2.1
Changed lines of the file:
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@@
 <part name="P1" library="_c2h" deviceset="PAD" device="NORMAL" value="GND"/>
 <part name="BAT2" library="edeca.net-v5" deviceset="BATT-CR123A" device="" value="CR123A"/>
-<part name="P2" library="_c2h" deviceset="PAD" device="NORMAL"/>
-<part name="P3" library="_c2h" deviceset="PAD" device="NORMAL"/>
 <part name="U$6" library="_c2h" deviceset="ARDUINO_PRO_MINI" device=""/>
 <part name="RGB" library="_c2h" deviceset="RGBLED_CA" device="STRAIGHT" value="RGBLED"/>
@@
 <attribute name="VALUE" x="36.195" y="139.7" size="1.778" layer="96" rot="R90"/>
 </instance>
-<instance part="P2" gate="G$1" x="46.355" y="51.435"/>
-<instance part="P3" gate="G$1" x="46.355" y="48.895"/>
 <instance part="U$6" gate="G$1" x="159.385" y="132.715"/>
 <instance part="RGB" gate="G$1" x="119.38" y="145.415" rot="R270"/>
@@
 </segment>
 <segment>
-<wire x1="61.595" y1="48.895" x2="46.355" y2="48.895" width="0.1524" layer="91"/>
-<junction x="46.355" y="48.895"/>
-<pinref part="P3" gate="G$1" pin="1"/>
-<wire x1="46.355" y1="48.895" x2="42.545" y2="48.895" width="0.1524" layer="91"/>
-<label x="48.895" y="48.895" size="1.778" layer="95"/>
+<wire x1="177.8" y1="112.395" x2="172.085" y2="112.395" width="0.1524" layer="91"/>
+<pinref part="U$6" gate="G$1" pin="A5-1"/>
+<junction x="172.085" y="112.395"/>
+<label x="173.99" y="112.395" size="1.778" layer="95"/>
 </segment>
 </net>
@@
 </segment>
 <segment>
-<wire x1="62.23" y1="51.435" x2="46.355" y2="51.435" width="0.1524" layer="91"/>
-<junction x="46.355" y="51.435"/>
-<pinref part="P2" gate="G$1" pin="1"/>
-<wire x1="46.355" y1="51.435" x2="42.545" y2="51.435" width="0.1524" layer="91"/>
-<label x="48.895" y="51.435" size="1.778" layer="95"/>
+<wire x1="177.8" y1="114.935" x2="172.085" y2="114.935" width="0.1524" layer="91"/>
+<pinref part="U$6" gate="G$1" pin="A4-1"/>
+<junction x="172.085" y="114.935"/>
+<label x="173.99" y="114.935" size="1.778" layer="95"/>
 </segment>
 </net>
