File: Mini-Lora.brd (EAGLE design)
At the start: 68.8 x 25.7 mm, 25 parts, among them P1 GND, P2 PADNORMAL, P3 PADNORMAL, P4 PADNORMAL, U1 24AA02E64T

Commit message: Bump to V1.1a
Parts:
- removed P2, P3: PADNORMAL, _c2h:PAD
Connections:
- net SCL: now also U$6.A5-1; no longer P3.1
- net SDA: now also U$6.A4-1; no longer P2.1
Routing:
- net SDA: track 26.4 -> 53.8 mm
- net SCL: track 25.5 -> 40.0 mm
- net 3V3: track 140.5 -> 141.3 mm
- net GND: vias 30 -> 31
Other:
- board text added: "Mini-Lora V1.1a"
- board text added: "V1.1a"
- board text removed: "Mini-Lora V1.1"
- board text removed: "V1.1"
Changed lines of the file:
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@@
 <grid distance="25" unitdist="mil" unit="mil" style="dots" multiple="1" display="yes" altdistance="5" altunitdist="mil" altunit="mil"/>
 <layers>
-<layer number="1" name="Top" color="4" fill="1" visible="no" active="yes"/>
+<layer number="1" name="Top" color="4" fill="1" visible="yes" active="yes"/>
 <layer number="2" name="Route2" color="1" fill="3" visible="no" active="no"/>
 <layer number="3" name="Route3" color="4" fill="3" visible="no" active="no"/>
 <layer number="14" name="Route14" color="1" fill="6" visible="no" active="no"/>
 <layer number="15" name="Route15" color="4" fill="6" visible="no" active="no"/>
-<layer number="16" name="Bottom" color="1" fill="1" visible="no" active="yes"/>
+<layer number="16" name="Bottom" color="1" fill="1" visible="yes" active="yes"/>
 <layer number="17" name="Pads" color="2" fill="1" visible="yes" active="yes"/>
 <layer number="18" name="Vias" color="2" fill="1" visible="yes" active="yes"/>
-<layer number="19" name="Unrouted" color="13" fill="1" visible="yes" active="yes"/>
+<layer number="19" name="Unrouted" color="6" fill="1" visible="yes" active="yes"/>
 <layer number="20" name="Dimension" color="15" fill="1" visible="yes" active="yes"/>
 <layer number="21" name="tPlace" color="7" fill="1" visible="yes" active="yes"/>
@@
 <layer number="25" name="tNames" color="7" fill="1" visible="yes" active="yes"/>
 <layer number="26" name="bNames" color="3" fill="1" visible="yes" active="yes"/>
-<layer number="27" name="tValues" color="7" fill="1" visible="yes" active="yes"/>
-<layer number="28" name="bValues" color="3" fill="1" visible="yes" active="yes"/>
+<layer number="27" name="tValues" color="48" fill="1" visible="yes" active="yes"/>
+<layer number="28" name="bValues" color="40" fill="1" visible="yes" active="yes"/>
 <layer number="29" name="tStop" color="7" fill="3" visible="yes" active="yes"/>
 <layer number="30" name="bStop" color="7" fill="6" visible="yes" active="yes"/>
@@
 <layer number="49" name="Reference" color="7" fill="1" visible="yes" active="yes"/>
 <layer number="50" name="dxf" color="7" fill="1" visible="no" active="no"/>
-<layer number="51" name="tDocu" color="7" fill="1" visible="yes" active="yes"/>
+<layer number="51" name="tDocu" color="6" fill="1" visible="yes" active="yes"/>
 <layer number="52" name="bDocu" color="3" fill="1" visible="yes" active="yes"/>
 <layer number="53" name="tGND_GNDA" color="7" fill="9" visible="no" active="no"/>
@@
 <text x="33.64975" y="10.257" size="0.889" layer="26" font="vector" ratio="15" rot="MR90">GND</text>
 <text x="33.64975" y="7.717" size="0.889" layer="26" font="vector" ratio="15" rot="MR90">3V3</text>
-<text x="52.60975" y="1.778" size="1.6764" layer="26" font="vector" ratio="15" rot="MR180" align="center">Mini-Lora V1.1</text>
+<text x="52.60975" y="1.778" size="1.6764" layer="26" font="vector" ratio="15" rot="MR180" align="center">Mini-Lora V1.1a</text>
 <text x="22.57425" y="20.60575" size="1.6764" layer="25" font="vector" ratio="15" align="center">Mini-Lora</text>
 <text x="23.23925" y="6.02725" size="1.27" layer="26" font="vector" ratio="15" rot="MR0">RFM95</text>
@@
 <text x="62.22475" y="12.6065" size="1.4224" layer="25" font="vector" ratio="15" rot="R90" align="center">GND</text>
 <text x="7.86875" y="12.8605" size="1.4224" layer="25" font="vector" ratio="15" rot="R90" align="center">3V3</text>
-<text x="29.81325" y="1.55575" size="1.6764" layer="25" font="vector" ratio="15" align="center">V1.1</text>
+<text x="29.81325" y="1.55575" size="1.6764" layer="25" font="vector" ratio="15" align="center">V1.1a</text>
 <text x="20.0025" y="23.59025" size="0.889" layer="26" font="vector" ratio="15" rot="MR90" align="center">GND</text>
 <text x="25.8445" y="23.59025" size="0.889" layer="26" font="vector" ratio="15" rot="MR90" align="center">3V3</text>
@@
 <element name="BAT2" library="edeca.net-v5" package="KEYSTONE-2/3A" value="CR123A" x="30.861" y="12.7" smashed="yes" rot="MR270"/>
 <element name="U$1" library="_c2h" package="PAD-JUMPER-SWAP" value="PAD-JUMPER-SWAPSWAP" x="38.735" y="10.16" smashed="yes" rot="MR180"/>
-<element name="P2" library="_c2h" package="PAD" value="PADNORMAL" x="35.56" y="16.51"/>
-<element name="P3" library="_c2h" package="PAD" value="PADNORMAL" x="35.56" y="13.97" smashed="yes"/>
 <element name="U$6" library="_c2h" package="ARDUINO_PRO_MINI" value="ARDUINO_PRO_MINI" x="50.8" y="12.7" smashed="yes" rot="R270"/>
 <element name="RGB" library="_c2h" package="LED5MMRGB_ST" value="RGBLED" x="11.811" y="3.556" smashed="yes" rot="R270">
@@
 <contactref element="BAT1" pad="GND@1"/>
 <via x="33.655" y="4.445" extent="1-16" drill="0.3556" diameter="0.7112"/>
-<via x="44.7675" y="15.24" extent="1-16" drill="0.3556" diameter="0.7112"/>
+<via x="44.3865" y="15.24" extent="1-16" drill="0.3556" diameter="0.7112"/>
 <via x="45.4025" y="8.255" extent="1-16" drill="0.3556" diameter="0.7112"/>
 <via x="66.421" y="17.7165" extent="1-16" drill="0.3556" diameter="0.7112"/>
@@
 <contactref element="U$6" pad="4"/>
 <via x="37.7825" y="16.764" extent="1-16" drill="0.3556" diameter="0.7112"/>
+<via x="44.3865" y="11.938" extent="1-16" drill="0.3556" diameter="0.7112"/>
 </signal>
 <signal name="SCL">
@@
 <contactref element="I2C" pad="3"/>
 <contactref element="U1" pad="1"/>
-<contactref element="P3" pad="1"/>
 <contactref element="U$6" pad="A5-0"/>
 <wire x1="42.7101" y1="12.1412" x2="42.7101" y2="11.5951" width="0.3048" layer="1"/>
@@
 <wire x1="27.305" y1="7.62" x2="28.21" y2="6.715" width="0.3048" layer="1"/>
 <wire x1="29.21" y1="6.715" x2="28.21" y2="6.715" width="0.3048" layer="1"/>
+<contactref element="U$6" pad="A5-1"/>
+<wire x1="54.76875" y1="7.9375" x2="54.76875" y2="8.73125" width="0.3048" layer="1"/>
+<wire x1="54.76875" y1="8.73125" x2="53.975" y2="9.525" width="0.3048" layer="1"/>
+<wire x1="53.975" y1="9.525" x2="43.18" y2="9.525" width="0.3048" layer="1"/>
+<wire x1="43.18" y1="9.525" x2="41.91" y2="10.795" width="0.3048" layer="1"/>
 </signal>
 <signal name="SDA">
@@
 <wire x1="32.39135" y1="16.51" x2="32.6136" y2="16.51" width="0.3048" layer="1"/>
 <wire x1="42.6593" y1="13.97" x2="42.7101" y2="14.0208" width="0.3048" layer="1"/>
-<contactref element="P2" pad="1"/>
 <wire x1="35.56" y1="16.51" x2="39.0525" y2="13.0175" width="0.3048" layer="1"/>
 <wire x1="32.39135" y1="16.51" x2="35.56" y2="16.51" width="0.3048" layer="1"/>
@@
 <wire x1="26.035" y1="12.7" x2="29.845" y2="16.51" width="0.3048" layer="1"/>
 <wire x1="29.845" y1="16.51" x2="32.39135" y2="16.51" width="0.3048" layer="1"/>
+<contactref element="U$6" pad="A4-1"/>
+<wire x1="52.22875" y1="7.9375" x2="52.22875" y2="7.46125" width="0.3048" layer="1"/>
+<wire x1="52.22875" y1="7.46125" x2="53.086" y2="6.604" width="0.3048" layer="1"/>
+<wire x1="53.086" y1="6.604" x2="54.102" y2="6.604" width="0.3048" layer="1"/>
+<wire x1="54.102" y1="6.604" x2="54.356" y2="6.35" width="0.3048" layer="1"/>
+<wire x1="54.356" y1="6.35" x2="55.372" y2="6.35" width="0.3048" layer="1"/>
+<wire x1="55.372" y1="6.35" x2="56.769" y2="7.747" width="0.3048" layer="1"/>
+<wire x1="44.45" y1="13.97" x2="42.7609" y2="13.97" width="0.3048" layer="1"/>
+<wire x1="42.7609" y1="13.97" x2="42.7101" y2="14.0208" width="0.3048" layer="1"/>
+<wire x1="56.769" y1="7.747" x2="56.769" y2="14.351" width="0.3048" layer="1"/>
+<wire x1="56.769" y1="14.351" x2="56.134" y2="14.986" width="0.3048" layer="1"/>
+<wire x1="56.134" y1="14.986" x2="45.466" y2="14.986" width="0.3048" layer="1"/>
+<wire x1="45.466" y1="14.986" x2="44.45" y2="13.97" width="0.3048" layer="1"/>
 </signal>
 <signal name="SCK">
@@
 <wire x1="53.34" y1="15.875" x2="52.07" y2="14.605" width="0.6096" layer="16"/>
 <wire x1="52.07" y1="14.605" x2="52.07" y2="11.43" width="0.6096" layer="16"/>
-<wire x1="52.07" y1="11.43" x2="50.8" y2="10.16" width="0.6096" layer="16"/>
-<wire x1="50.8" y1="10.16" x2="42.8625" y2="10.16" width="0.6096" layer="16"/>
 <wire x1="52.705" y1="16.51" x2="53.34" y2="15.875" width="0.4064" layer="1"/>
 <via x="53.34" y="15.875" extent="1-16" drill="0.3556" diameter="0.7112"/>
@@
 <contactref element="U$1" pad="44"/>
 <wire x1="29.591" y1="7.239" x2="31.115" y2="7.239" width="0.6096" layer="16"/>
-<wire x1="31.115" y1="7.239" x2="39.9415" y2="7.239" width="0.6096" layer="16"/>
-<wire x1="39.9415" y1="7.239" x2="41.9735" y2="9.271" width="0.6096" layer="16"/>
-<wire x1="41.9735" y1="9.271" x2="42.8625" y2="10.16" width="0.6096" layer="16"/>
-<wire x1="39.6113" y1="9.271" x2="41.9735" y2="9.271" width="0.6096" layer="16"/>
+<wire x1="31.115" y1="7.239" x2="41.91" y2="7.239" width="0.6096" layer="16"/>
+<wire x1="41.91" y1="7.239" x2="47.879" y2="7.239" width="0.6096" layer="16"/>
 <wire x1="39.6113" y1="11.049" x2="39.6113" y2="9.271" width="0.6096" layer="16"/>
 <wire x1="26.019" y1="4.699" x2="26.035" y2="4.715" width="0.4064" layer="1"/>
@@
 <wire x1="9.525" y1="5.08" x2="10.287" y2="4.318" width="0.4064" layer="16"/>
 <wire x1="11.7951" y1="4.318" x2="10.287" y2="4.318" width="0.4064" layer="16"/>
+<wire x1="52.07" y1="11.43" x2="47.879" y2="7.239" width="0.6096" layer="16"/>
+<wire x1="39.6113" y1="9.271" x2="39.878" y2="9.271" width="0.6096" layer="16"/>
+<wire x1="39.878" y1="9.271" x2="41.91" y2="7.239" width="0.6096" layer="16"/>
 </signal>
 <signal name="SS">

Commit message: Bump to V1.2
Parts:
- removed U$3: (no value), _c2h:LOGO_CH2I_75MM
- added C3: 100nF, _c2h:0805-CAP
- added P2, P3: PADNORMAL, _c2h-MacBook Pro de Charles-Henri:PAD
- added R7: 100K, _c2h:0805-RES
- added R9: 47K, _c2h:1206-RES
- added U$2: (no value), _c2h:LOGO_C2I_015
- added U2: TPL5110, microbuilder:SOT23-6
- added WAKE: WAKE, Switch-2016:SW4-SMD-4.2X3.2X2.5MM
- R4: value 220 -> 680
- R5: value 100 -> 470
- R6: value 100 -> 1.5K
- U$6: value ARDUINO_PRO_MINI -> ARDUINO MINI 3.3V 8Mhz
- moved R3 32.1 mm to (50.8, 17.4), turned to 90 degrees
- moved R2 3.59 mm to (31.8, 3.17)
- moved C1 3.18 mm to (37.8, 15.6), turned to 270 degrees
- moved R1 3.18 mm to (27.9, 3.17)
- moved BTN 3.11 mm to (17.1, 15.9), turned to 180 degrees
- moved U1 2.84 mm to (42.6, 15.6)
- moved R5 2.44 mm to (24.8, 4.19), turned to 180 degrees
- moved R6 2.16 mm to (20.6, 4.19), turned to 180 degrees
- moved R4 1.65 mm to (16.5, 4.19), turned to 180 degrees
Connections:
- removed net A1: U$6.18
- removed net A2: U$6.19
- new net DELAY: P2.1, R9.2, U2.3, WAKE.3
- new net DONE: R7.2, U$6.18, U2.4
- new net DRVN: U$6.19, U2.5
- net 3V3: now also C3.1, U2.1, U2.6, WAKE.2
- net GND: now also C3.2, P3.1, R7.1, R9.1, U2.2
Routing:
- net 3V3: track 141.3 -> 171.9 mm
- net DELAY: track 0.00 -> 27.7 mm, vias 0 -> 2
- net DRVN: track 0.00 -> 10.2 mm
- net DONE: track 0.00 -> 7.33 mm
- net D3: track 41.0 -> 35.9 mm
- net GND: track 1.78 -> 3.93 mm, vias 31 -> 35
- net RED: track 28.2 -> 30.3 mm
- net BLUE: track 34.2 -> 32.2 mm
- net SS: track 17.0 -> 18.8 mm
- net SCL: track 40.0 -> 39.3 mm
- net LB: track 12.5 -> 13.2 mm
Other:
- board text added: "24AA02"
- board text added: "BLU"
- board text added: "BTN"
- board text added: "D5/B"
- board text added: "D6/G"
- board text added: "D9/R"
- board text added: "GRN"
- board text added: "Mini-Lora V1.2"
- board text added: "RED"
- board text added: "RES"
- board text added: "TPL"
- board text added: "V1.2"
- board text added: "done"
- board text added: "drvn"
- board text removed: "A0"
- board text removed: "A1"
- board text removed: "A2"
- board text removed: "BTN D3"
- board text removed: "D5"
- board text removed: "D5 B"
- board text removed: "D6"
- board text removed: "D6 G"
- board text removed: "D9"
- board text removed: "D9 R"
- board text removed: "Mini-Lora V1.1a"
- board text removed: "V1.1a"
