File: Mini-Lora.sch (EAGLE design)
At the start: 23 parts, among them P1 GND, P2 PADNORMAL, P3 PADNORMAL, P4 PADNORMAL, U1 24AA02E64T

Commit message: Bump to V1.1a
Parts:
- removed P2, P3: PADNORMAL, _c2h:PADNORMAL
Connections:
- net SCL: now also U$6.A5-1; no longer P3.1
- net SDA: now also U$6.A4-1; no longer P2.1
Changed lines of the file:
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@@
 <part name="NAME" library="SparkFun-Aesthetics" deviceset="FRAME-A4L" device="" value="Value">
 <attribute name="CNAME" value="Arduino Mini Lora Shield"/>
-<attribute name="CREVISION" value="1.1"/>
+<attribute name="CREVISION" value="1.1a"/>
 <attribute name="DESIGNER" value="Charles-Henri Hallard"/>
 </part>
@@
 <part name="+3V3" library="supply1" deviceset="+3V3" device="" value="3V3"/>
 <part name="GND1" library="supply1" deviceset="GND" device=""/>
-<part name="P2" library="_c2h" deviceset="PAD" device="NORMAL"/>
-<part name="P3" library="_c2h" deviceset="PAD" device="NORMAL"/>
 <part name="U$6" library="_c2h" deviceset="ARDUINO_PRO_MINI" device=""/>
 <part name="RGB" library="_c2h" deviceset="RGBLED_CA" device="STRAIGHT" value="RGBLED"/>
@@
 </instance>
 <instance part="GND1" gate="1" x="77.47" y="51.435"/>
-<instance part="P2" gate="G$1" x="46.355" y="51.435"/>
-<instance part="P3" gate="G$1" x="46.355" y="48.895"/>
 <instance part="U$6" gate="G$1" x="159.385" y="132.715"/>
 <instance part="RGB" gate="G$1" x="119.38" y="145.415" rot="R270"/>
@@
 </segment>
 <segment>
-<wire x1="61.595" y1="48.895" x2="46.355" y2="48.895" width="0.1524" layer="91"/>
-<junction x="46.355" y="48.895"/>
-<pinref part="P3" gate="G$1" pin="1"/>
-<wire x1="46.355" y1="48.895" x2="42.545" y2="48.895" width="0.1524" layer="91"/>
-<label x="48.895" y="48.895" size="1.778" layer="95"/>
+<wire x1="177.8" y1="112.395" x2="172.085" y2="112.395" width="0.1524" layer="91"/>
+<pinref part="U$6" gate="G$1" pin="A5-1"/>
+<junction x="172.085" y="112.395"/>
 </segment>
 </net>
@@
 </segment>
 <segment>
-<wire x1="62.23" y1="51.435" x2="46.355" y2="51.435" width="0.1524" layer="91"/>
-<junction x="46.355" y="51.435"/>
-<pinref part="P2" gate="G$1" pin="1"/>
-<wire x1="46.355" y1="51.435" x2="42.545" y2="51.435" width="0.1524" layer="91"/>
-<label x="48.895" y="51.435" size="1.778" layer="95"/>
+<wire x1="177.8" y1="114.935" x2="172.085" y2="114.935" width="0.1524" layer="91"/>
+<pinref part="U$6" gate="G$1" pin="A4-1"/>
+<junction x="172.085" y="114.935"/>
 </segment>
 </net>

Commit message: Bump to V1.2
Parts:
- added C3: 100nF, _c2h:CAP0805-CAP
- added P2, P3: PADNORMAL, _c2h-MacBook Pro de Charles-Henri:PADNORMAL
- added R7: 100K, _c2h:RESISTOR0805-RES
- added R9: 47K, _c2h:RESISTOR'1206-RES''
- added U2: TPL5110, microbuilder:TPL5111
- added WAKE: WAKE, Switch-2016:SMD-BUTTON-TOP-DHT-4235A(4P-4.2X3.2MM)
- R4: value 220 -> 680
- R5: value 100 -> 470
- R6: value 100 -> 1.5K
- U$6: value ARDUINO_PRO_MINI -> ARDUINO MINI 3.3V 8Mhz
Connections:
- removed net A1: U$6.A1
- removed net A2: U$6.A2
- new net DELAY: P2.1, R9.2, U2.DELAY, WAKE.B0
- new net DONE: R7.2, U$6.A1, U2.DONE
- new net DRVN: U$6.A2, U2.DRVN
- net 3V3: now also C3.1, U2.EN, U2.VDD, WAKE.A1
- net GND: now also C3.2, P3.1, R7.1, R9.1, U2.GND
Other:
- note added: "Arduino Mini"
- note added: "Batteries connectors"
- note added: "Button and Low Power"
- note added: "For Low Power Remove Regulator from board Remove Power Led from board"
- note added: "I2C and DEVEUI"
- note added: "LoRa"
- note added: "RGB Led resistors choosen after testing luminosity on 3V3 board with my stocked RGB Leds. Light is same level from Red, Green and Blue with these values"
- note added: "Wake Time interval relation with R9 170K 2 hours 120K ~1 hour 100K ~35 min 47K ~6 min"
- moved on the sheet: BAT1, BAT2, BAT3, BTN, C1, C2, I2C, R1, R2, R3, R4, R5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
